Commit message: Parametrize husky wheel friction and reduce right Husky has issues turning in place. This is currently an open issue many are experiencing with the husky. No official solution as of yet. One user noted that the right wheel friction seems greater than the left wheels friction. Solution is to reduce friction of both right wheels. Seems to alleviate the issue: https://github.com/husky/husky/issues/120

File: mipp_description/urdf/husky.urdf.xacro (robot description, xacro)
@@ -103,14 +103,14 @@
   </gazebo>
   <!-- Husky wheel macros -->
-  <xacro:husky_wheel wheel_prefix="front_left">
+  <xacro:husky_wheel wheel_prefix="front_left" mu1="1.0" mu2="1.0">
     <origin xyz="${wheelbase/2} ${track/2} ${wheel_vertical_offset}" rpy="0 0 0" />
   </xacro:husky_wheel>
-  <xacro:husky_wheel wheel_prefix="front_right">
+  <xacro:husky_wheel wheel_prefix="front_right" mu1="0.5" mu2="0.5">
     <origin xyz="${wheelbase/2} ${-track/2} ${wheel_vertical_offset}" rpy="0 0 0" />
   </xacro:husky_wheel>
-  <xacro:husky_wheel wheel_prefix="rear_left">
+  <xacro:husky_wheel wheel_prefix="rear_left" mu1="1.0" mu2="1.0">
     <origin xyz="${-wheelbase/2} ${track/2} ${wheel_vertical_offset}" rpy="0 0 0" />
   </xacro:husky_wheel>
-  <xacro:husky_wheel wheel_prefix="rear_right">
+  <xacro:husky_wheel wheel_prefix="rear_right" mu1="0.5" mu2="0.5">
     <origin xyz="${-wheelbase/2} ${-track/2} ${wheel_vertical_offset}" rpy="0 0 0" />
   </xacro:husky_wheel>

File: mipp_description/urdf/wheel.urdf.xacro (robot description, xacro)
@@ -22,5 +22,5 @@
 -->
 <robot xmlns:xacro="http://ros.org/wiki/xacro" name="husky_wheel">
-	<xacro:macro name="husky_wheel" params="wheel_prefix *joint_pose">
+	<xacro:macro name="husky_wheel" params="wheel_prefix mu1 mu2 *joint_pose">
 		<link name="${wheel_prefix}_wheel_link">
 			<inertial>
@@ -43,6 +43,6 @@
 		</link>
 		<gazebo reference="${wheel_prefix}_wheel_link">
-			<mu1 value="1.0"/>
-			<mu2 value="1.0"/>
+			<mu1 value="${mu1}"/>
+			<mu2 value="${mu2}"/>
 			<kp value="10000000.0" />
 			<kd value="1.0" />
