Commit message: Give up on using smart pointers.

File: mipp_description/urdf/accessories/extras.urdf.xacro (robot description, xacro)
@@ -14,11 +14,19 @@
         </plugin>
     </gazebo>
-    <!-- Velodyne 3D Lidar (mounted on sensor arch)-->
+    <!-- Sensor arch -->
     <xacro:sensor_arch prefix="" parent="top_plate_link">
         <origin xyz="0 0 0.51" rpy="0 0 0"/>
     </xacro:sensor_arch>
+    <!-- Velodyne 3D Lidar (mounted on sensor arch) -->
     <xacro:include filename="$(find velodyne_description)/urdf/VLP-16.urdf.xacro"/>
     <VLP-16 parent="sensor_arch_mount_link" name="velodyne" topic="gazebo/velodyne_points" hz="5" samples="440">
         <origin xyz="0 0 0" rpy="0 0 0" />
     </VLP-16>
+    <!-- Camera (mounted on sensor arch)
+    <joint name="kinect_frame_joint" type="fixed">
+      <origin xyz="0 0 -0.05" rpy="0 0 0" />
+      <parent link="sensor_arch_mount_link"/>
+      <child link="camera_link"/>
+    </joint>
+    <xacro:kinect_camera prefix="camera" robot_namespace="/"/>-->
 </robot>

Commit message: Add an overhead camera

File: mipp_description/urdf/accessories/extras.urdf.xacro (robot description, xacro)
@@ -22,3 +22,9 @@
         <origin xyz="0 0 0" rpy="0 0 0" />
     </VLP-16>
+    <joint name="kinect_frame_joint" type="fixed">
+        <origin xyz="-7.0 0 7.00" rpy="0 0.785 0.0"/>
+        <parent link="sensor_arch_mount_link"/>
+        <child link="overhead_camera_link"/>
+    </joint>
+    <xacro:kinect_camera prefix="overhead_camera" robot_namespace="$(arg robot_namespace)"/>
 </robot>

File: mipp_description/urdf/accessories/kinect_camera.urdf.xacro (robot description, xacro)
@@ -32,5 +32,5 @@
       <origin xyz="0 0 0" rpy="0 0 0"/>
       <visual>
-        <origin xyz="0 0 0" rpy="0 0 ${M_PI/2}"/>
+        <origin xyz="0 0 100" rpy="0 0 ${M_PI/2}"/>
         <geometry>
           <mesh filename="package://husky_description/meshes/accessories/kinect.dae" />
@@ -54,13 +54,13 @@
         <update_rate>20.0</update_rate>
         <camera>
-          <horizontal_fov>${60.0*M_PI/180.0}</horizontal_fov>
+          <horizontal_fov>${90.0*M_PI/180.0}</horizontal_fov>
           <image>
             <format>R8G8B8</format>
-            <width>640</width>
+            <width>960</width>
             <height>480</height>
           </image>
           <clip>
             <near>0.05</near>
-            <far>8.0</far>
+            <far>20.0</far>
           </clip>
         </camera>
